File: hardware/led_sign_2020.kicad_pcb (KiCad board)
At the start: 2 copper layers, 25 parts, among them Q1 STD26P3LLH6, U1 ESP32-DevKitC, U2 MC74VHC1GT125, U3 MC74VHC1GT125, U4 MAX17601, U5 MAX17601, U6 MAX17601, U7 MAX17601

Commit message: footprints
Parts:
- added C8: 0.1uF, Capacitor_SMD:C_0805_2012Metric, F.Cu at (79.2, 20.8)
- added D4: D_Zener, Diode_SMD:D_0805_2012Metric, F.Cu at (64.0, 39.6)
- moved R5 64.3 mm to (53.8, 41.1), turned to 90 degrees
- moved D2 49.8 mm to (57.9, 49.8)
- moved U7 26.6 mm to (105.2, 45.2)
- moved U4 22.9 mm to (105.2, 20.3)
- moved C2 20.6 mm to (98.6, 76.2)
- moved U6 19.0 mm to (105.2, 36.7)
- moved U5 18.8 mm to (105.2, 28.4)
- moved D3 18.4 mm to (107.8, 68.1)
- moved C6 13.3 mm to (122.5, 75.0)
- moved R1 12.4 mm to (132.7, 50.8)
- moved JP1 9.58 mm to (42.2, 54.4)
- moved C1 8.27 mm to (124.5, 41.1)
- moved JP2 7.62 mm to (42.7, 39.6)
- moved Q1 7.15 mm to (51.3, 29.9)
- moved U1 6.85 mm to (80.3, 57.9)
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Connections:
- net Net-(U1-Pad36) renamed /CDATA
- net Net-(U1-Pad37) renamed /CCLK
- C2 pad 1: +5V -> /C5V
- C3 pad 1: Net-(C3-Pad1) -> GND
- C3 pad 2: GND -> +5V
- C4 pad 1: +5V -> GND
- C4 pad 2: GND -> +5V
- C5 pad 1: +5V -> GND
- C5 pad 2: GND -> +5V
- C6 pad 1: +5V -> GND
- C6 pad 2: GND -> +5V
- JP1 pad 2: Net-(C3-Pad1) -> /C5V
- R1 pad 2: Net-(R1-Pad2) -> /EN
- R3 pad 2: Net-(C3-Pad1) -> /C5V
- R4 pad 2: Net-(R1-Pad2) -> /EN
- U1 pad 12: (no net) -> /C3
- U1 pad 13: (no net) -> /C1
- U1 pad 15: (no net) -> /C2
- U1 pad 19: Net-(C3-Pad1) -> /C5V
- U1 pad 23: (no net) -> /C4
- U1 pad 27: (no net) -> /C5
- U1 pad 28: (no net) -> /C6
- U1 pad 30: (no net) -> /C7
- U4 pad 2: (no net) -> /C1
- U4 pad 3: (no net) -> GND
- U4 pad 4: (no net) -> /C2
- U4 pad 8: (no net) -> /EN
- U5 pad 2: (no net) -> /C3
- U5 pad 3: (no net) -> GND
- U5 pad 4: (no net) -> /C4
- U5 pad 6: (no net) -> +5V
- U5 pad 8: (no net) -> /EN
- U6 pad 2: (no net) -> /C5
- U6 pad 3: (no net) -> GND
- U6 pad 4: (no net) -> /C6
- U6 pad 6: (no net) -> +5V
- U6 pad 8: (no net) -> /EN
- U7 pad 2: (no net) -> /C7
- U7 pad 3: (no net) -> GND
- U7 pad 6: (no net) -> +5V

Commit message: routing pcb
Parts:
- removed the C7 at (132.1, 31.3)
- added C1: CP1, Capacitor_THT:CP_Radial_D10.0mm_P5.00mm, F.Cu at (82.5, 113.5)
- added CONN1: LED_sign_connection, Connector_JST:JST_XH_B12B-XH-A_1x12_P2.50mm_Vertical, F.Cu at (114.0, 62.5)
- added PWR_CONN1: Conn_01x02_Male, Connector_JST:JST_XH_B2B-XH-A_1x02_P2.50mm_Vertical, F.Cu at (130.5, 61.5)
- JP1: value Jumper_2_Open -> ESP32_5V
- JP2: value Jumper_2_Open -> prot_short
- moved U4 99.2 mm to (132.7, 115.7), turned to 270 degrees
- moved Q1 95.4 mm to (133.5, 78.3)
- moved R5 93.8 mm to (136.0, 86.4)
- moved C8 91.7 mm to (132.5, 95.5), turned to 90 degrees
- moved U5 89.0 mm to (123.5, 115.5), turned to 270 degrees
- moved JP2 84.4 mm to (124.5, 60.5)
- moved D4 82.2 mm to (131.5, 86.5), turned to 90 degrees
- moved U6 79.3 mm to (114.0, 115.5), turned to 270 degrees
- moved JP1 78.1 mm to (120.0, 60.5)
- moved D2 71.1 mm to (125.9, 70.5), turned to 180 degrees
- moved C3 70.1 mm to (133.6, 109.0), turned to 180 degrees
- moved U7 69.9 mm to (104.5, 115.2), turned to 270 degrees
- moved C4 69.4 mm to (124.5, 109.0), turned to 180 degrees
- moved D1 68.7 mm to (125.9, 68.0), turned to 180 degrees
- moved C7 59.3 mm to (132.5, 100.0), turned to 90 degrees
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- renumbered C1 to C7
Connections:
- U2 pad 4: (no net) -> /DATA
- U3 pad 4: (no net) -> /CLK
- U4 pad 5: (no net) -> /R2
- U4 pad 7: (no net) -> /R1
- U5 pad 5: (no net) -> /R4
- U5 pad 7: (no net) -> /R3
- U6 pad 5: (no net) -> /R6
- U6 pad 7: (no net) -> /R5
- U7 pad 7: (no net) -> /R7
Routing:
- net +5V: track 0.00 -> 226.5 mm, vias 0 -> 2
- net GND: track 0.00 -> 190.6 mm, vias 0 -> 4
- net /C5V: track 0.00 -> 52.7 mm, vias 0 -> 1
- net Net-(JP2-Pad1): track 0.00 -> 37.5 mm
- net Net-(D4-Pad2): track 0.00 -> 7.72 mm
- net Net-(D3-Pad2): track 0.00 -> 2.52 mm
- net Net-(D2-Pad2): track 0.00 -> 2.00 mm
- net Net-(D1-Pad2): track 0.00 -> 2.00 mm
- net (no net): vias 0 -> 6
Other:
- board outline added: 70 x 100 mm

Commit message: board layout
Parts:
- moved C1 58.0 mm to (138.3, 97.6), turned to 180 degrees
- moved U4 51.1 mm to (107.2, 71.4), turned to 90 degrees
- moved U5 50.4 mm to (99.1, 71.4), turned to 90 degrees
- moved U6 49.8 mm to (91.0, 71.4), turned to 90 degrees
- moved U7 48.8 mm to (82.9, 71.3), turned to 90 degrees
- moved C3 48.4 mm to (103.1, 71.3), turned to 90 degrees
- moved C4 47.8 mm to (95.1, 71.3), turned to 90 degrees
- moved C5 46.5 mm to (87.0, 71.4), turned to 90 degrees
- moved C6 45.6 mm to (79.0, 71.4), turned to 90 degrees
- moved U2 34.9 mm to (113.1, 74.7)
- moved R1 31.7 mm to (126.2, 74.7), turned to 270 degrees
- moved C7 29.9 mm to (116.5, 74.7), turned to 270 degrees
- moved U3 25.6 mm to (122.0, 74.7)
- moved C8 25.0 mm to (118.6, 74.7), turned to 270 degrees
- moved C2 13.5 mm to (123.7, 115.6), turned to 180 degrees
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Routing:
- net /EN: track 0.00 -> 140.5 mm, vias 0 -> 12
- net GND: track 190.6 -> 315.6 mm, vias 4 -> 7
- net /CLK: track 0.00 -> 75.4 mm, vias 0 -> 2
- net /CCLK: track 0.00 -> 61.2 mm, vias 0 -> 2
- net /DATA: track 0.00 -> 57.6 mm, vias 0 -> 2
- net /C2: track 0.00 -> 55.2 mm, vias 0 -> 2
- net /C3: track 0.00 -> 52.4 mm, vias 0 -> 2
- net /C1: track 0.00 -> 49.8 mm, vias 0 -> 2
- net /CDATA: track 0.00 -> 48.8 mm, vias 0 -> 2
- net /C4: track 0.00 -> 36.7 mm, vias 0 -> 2
- net /C5: track 0.00 -> 34.0 mm, vias 0 -> 2
- net /C7: track 0.00 -> 30.6 mm, vias 0 -> 2
- net /C6: track 0.00 -> 27.4 mm, vias 0 -> 2
- net +5V: track 226.5 -> 205.6 mm
- net /C5V: track 52.7 -> 70.9 mm, vias 1 -> 2
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Other:
- board size 70 x 100 mm -> 70 x 70 mm
- board text added: "SilentRadio LED sign controller v2"
- board text added: "jason plumb :: noisybox.net"

Commit message: fix stray net
Other:
- board text added: "jason plumb :: noisybox.net - january 2021"
- board text removed: "jason plumb :: noisybox.net"

Commit message: beef up those power busses
Routing:
- net +5V: track 205.6 -> 208.8 mm
- net /R1: track 7.57 -> 9.53 mm
- net GND: track 315.6 -> 314.1 mm
- net /EN: track 140.5 -> 139.8 mm

Commit message: wip
Parts:
- moved JP1 69.1 mm to (125.4, 129.4), turned to 90 degrees
- moved D4 41.0 mm to (172.0, 80.1)
- moved Q1 41.0 mm to (174.0, 71.9)
- moved R5 41.0 mm to (176.5, 80.0)
- moved U7 29.3 mm to (112.2, 71.5)
- moved C6 29.3 mm to (108.3, 71.5)
- moved C7 29.0 mm to (120.6, 46.0)
- moved C8 29.0 mm to (122.7, 46.0)
- moved D1 29.0 mm to (130.0, 39.3)
- moved D2 29.0 mm to (130.0, 41.8)
- moved D3 29.0 mm to (121.2, 41.8)
- moved R2 29.0 mm to (126.2, 39.3)
- moved R3 29.0 mm to (126.0, 41.8)
- moved R4 29.0 mm to (121.2, 39.3)
- moved U2 29.0 mm to (117.2, 46.0)
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Routing:
- net GND: track 314.1 -> 146.1 mm
- net +5V: track 208.8 -> 100.6 mm, vias 2 -> 4
- net /EN: track 139.8 -> 55.1 mm, vias 12 -> 8
- net /CLK: track 75.4 -> 0.00 mm, vias 2 -> 0
- net /C5V: track 71.0 -> 0.00 mm, vias 2 -> 0
- net /CCLK: track 61.2 -> 0.00 mm, vias 2 -> 0
- net /DATA: track 57.6 -> 0.00 mm, vias 2 -> 0
- net /C2: track 55.2 -> 0.00 mm, vias 2 -> 0
- net /C3: track 52.4 -> 0.00 mm, vias 2 -> 0
- net /C1: track 49.8 -> 0.00 mm, vias 2 -> 0
- net /CDATA: track 48.8 -> 0.00 mm, vias 2 -> 0
- net /C4: track 36.7 -> 0.00 mm, vias 2 -> 0
- net /C5: track 34.0 -> 0.00 mm, vias 2 -> 0
- net /C7: track 30.6 -> 0.00 mm, vias 2 -> 0
- net /C6: track 27.4 -> 0.00 mm, vias 2 -> 0
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Other:
- board size 70 x 70 mm -> 70 x 86 mm

Commit message: reroute in progress
Parts:
- moved R5 51.2 mm to (125.3, 78.9), turned to 0 degrees
- moved R1 51.0 mm to (96.9, 84.5), turned to 180 degrees
- moved Q1 46.6 mm to (127.5, 71.7)
- moved D4 43.0 mm to (129.0, 78.9), turned to 180 degrees
- moved U3 30.3 mm to (117.7, 75.1)
- moved C8 29.3 mm to (120.8, 75.2)
- moved R2 25.1 mm to (123.3, 64.2), turned to 270 degrees
- moved R4 25.0 mm to (118.7, 64.2), turned to 270 degrees
- moved U2 23.5 mm to (117.6, 69.5)
- moved C7 23.5 mm to (120.8, 69.5)
- moved R3 23.0 mm to (121.0, 64.2), turned to 270 degrees
- moved D1 22.1 mm to (123.3, 60.4), turned to 270 degrees
- moved D2 20.7 mm to (121.0, 60.4), turned to 270 degrees
- moved D3 18.8 mm to (118.7, 60.4), turned to 270 degrees
- moved JP1 6.96 mm to (126.3, 122.5)
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Routing:
- net +5V: track 100.6 -> 236.5 mm
- net GND: track 146.1 -> 191.4 mm, vias 7 -> 5
- net /CLK: track 0.00 -> 18.5 mm, vias 0 -> 2
- net /DATA: track 0.00 -> 14.3 mm
- net /EN: track 55.1 -> 67.4 mm, vias 8 -> 9
- net Net-(JP2-Pad1): track 12.7 -> 15.2 mm
- net Net-(D4-Pad2): track 7.72 -> 5.34 mm
- net Net-(D3-Pad2): track 3.35 -> 1.95 mm
- net /C5V: track 0.00 -> 1.08 mm

Commit message: routed
Parts:
- moved C2 17.0 mm to (120.6, 116.8)
- moved U1 6.33 mm to (104.8, 99.5)
- moved JP1 5.89 mm to (127.3, 116.7), turned to 270 degrees
- moved R1 4.38 mm to (93.7, 81.5), turned to 0 degrees
Routing:
- net GND: track 191.4 -> 280.6 mm, vias 5 -> 8
- net /C5V: track 1.08 -> 65.2 mm
- net /C2: track 0.00 -> 61.4 mm
- net /C1: track 0.00 -> 57.7 mm
- net /C4: track 0.00 -> 50.2 mm
- net /C3: track 0.00 -> 50.1 mm, vias 0 -> 2
- net /CDATA: track 0.00 -> 44.1 mm, vias 0 -> 4
- net /CCLK: track 0.00 -> 42.2 mm, vias 0 -> 2
- net /C7: track 0.00 -> 27.9 mm
- net +5V: track 236.5 -> 260.8 mm, vias 4 -> 6
- net /C5: track 0.00 -> 23.3 mm
- net /C6: track 0.00 -> 11.9 mm
- net /EN: track 67.4 -> 79.0 mm
- net Net-(JP2-Pad1): track 15.2 -> 21.5 mm
- net /CLK: track 18.5 -> 19.2 mm
