File: hardware/led_sign_2020.sch (KiCad schematic (older format))
At the start: 29 parts, among them Q1 STD26P3LLH6, U1 ESP32-DevKitC, U2 MC74VHC1GT125, U3 MC74VHC1GT125, U4 MAX17601, U5 MAX17601, U6 MAX17601, U7 MAX17601

Commit message: footprint
Parts:
- D4: footprint Diode_SMD:D_0805_2012Metric -> Diode_SMD:D_SOD-123
Changed lines of the file:
@@
 F 0 "D4" V 3225 2100 50  0000 L CNN
 F 1 "D_Zener" V 3270 2330 50  0001 L CNN
-F 2 "Diode_SMD:D_0805_2012Metric" H 3225 2250 50  0001 C CNN
+F 2 "Diode_SMD:D_SOD-123" H 3225 2250 50  0001 C CNN
 F 3 "~" H 3225 2250 50  0001 C CNN
 	1    3225 2250
